Commit message: updating urdf

File: mycobot_client_2/models/elephant_description/mycobot_280_pi_simple.urdf (robot description, URDF)
Before this commit: robot myCobot_280, 10 links, 9 joints
Joints:
- joint joint2_to_joint1: origin xyz=0 0 0.13956 rpy=0 0 0 -> xyz=0 0 -0.13956 rpy=3.14 0 0

Commit message: updating pybullet

File: mycobot_client_2/models/elephant_description/mycobot_280_pi_simple.urdf (robot description, URDF)
Before this commit: robot myCobot_280, 10 links, 9 joints
Joints:
- joint joint2_to_joint1: origin xyz=0 0 -0.13956 rpy=3.14 0 0 -> xyz=0 0 0.13956 rpy=0 0 0
