Commit message: adding gripper

File: mycobot_client_2/models/elephant_description/mycobot_280_pi.urdf (robot description, URDF)
Before this commit: robot firefighter, 8 links, 7 joints
Links:
- added link gripper; collision cylinder length=0.3 radius=0.2; visual cylinder length=0.3 radius=0.2
Joints:
- added joint joint6output_to_gripper: type fixed, parent joint6_flange, child gripper, origin xyz=0 0 0.034 rpy=1.579 0 0

Commit message: updating gripper

File: mycobot_client_2/models/elephant_description/mycobot_280_pi.urdf (robot description, URDF)
Before this commit: robot firefighter, 9 links, 8 joints
Links:
- link gripper: geometry collision cylinder length=0.3 radius=0.1; visual cylinder length=0.3 radius=0.1

Commit message: trying just coordinate frame

File: mycobot_client_2/models/elephant_description/mycobot_280_pi.urdf (robot description, URDF)
Before this commit: robot firefighter, 9 links, 8 joints
Links:
- link gripper: geometry 
Joints:
- joint joint6output_to_gripper: origin xyz=0 0 0.034 rpy=1.579 0 0 -> xyz=0 0 0.2 rpy=0 0 0

Commit message: updating gripper location

File: mycobot_client_2/models/elephant_description/mycobot_280_pi.urdf (robot description, URDF)
Before this commit: robot firefighter, 9 links, 8 joints
Joints:
- joint joint6output_to_gripper: origin xyz=0 0 0.2 rpy=0 0 0 -> xyz=0 0 0.12 rpy=0 0 0

Commit message: updating urdf to account for z shift for g base and acryllic

File: mycobot_client_2/models/elephant_description/mycobot_280_pi.urdf (robot description, URDF)
Before this commit: robot firefighter, 9 links, 8 joints
Links:
- added link robot_base
Joints:
- added joint robot_base_to_g_base: type fixed, parent robot_base, child g_base, origin xyz=0 0 0.12 rpy=0 0 0

Commit message: updating urdf

File: mycobot_client_2/models/elephant_description/mycobot_280_pi.urdf (robot description, URDF)
Before this commit: robot firefighter, 10 links, 9 joints
Joints:
- joint joint6output_to_gripper: origin xyz=0 0 0.12 rpy=0 0 0 -> xyz=0 0 0.1 rpy=0 0 0
- joint robot_base_to_g_base: origin xyz=0 0 0.12 rpy=0 0 0 -> xyz=0 0 0.003 rpy=0 0 0

Commit message: adding gbase displacement

File: mycobot_client_2/models/elephant_description/mycobot_280_pi.urdf (robot description, URDF)
Before this commit: robot firefighter, 10 links, 9 joints
Joints:
- joint g_base_to_joint1: origin xyz=0 0 0 rpy=0 0 0 -> xyz=0 0 0.026 rpy=0 0 0

Commit message: updating G base

File: mycobot_client_2/models/elephant_description/mycobot_280_pi.urdf (robot description, URDF)
Before this commit: robot firefighter, 10 links, 9 joints
Links:
- link g_base: mass 0.2 -> None; geometry 

Commit message: adding simple urdf

File: mycobot_client_2/models/elephant_description/mycobot_280_pi.urdf (robot description, URDF)
Before this commit: robot firefighter, 10 links, 9 joints
Links:
- link g_base: mass None -> 0.2; geometry collision mesh filename=G_base_new.dae; visual mesh filename=G_base_new.dae

Commit message: flipping sign in urdf

File: mycobot_client_2/models/elephant_description/mycobot_280_pi.urdf (robot description, URDF)
Before this commit: robot firefighter, 10 links, 9 joints
Links:
- link g_base: mass 0.2 -> None; geometry 
Joints:
- joint g_base_to_joint1: origin xyz=0 0 0.026 rpy=0 0 0 -> xyz=0 0 0.026 rpy=3.141 0 0

Commit message: updating urdf

File: mycobot_client_2/models/elephant_description/mycobot_280_pi.urdf (robot description, URDF)
Before this commit: robot firefighter, 10 links, 9 joints
Joints:
- joint g_base_to_joint1: origin xyz=0 0 0.026 rpy=3.141 0 0 -> xyz=0 0 0.026 rpy=0 0 0
- joint joint2_to_joint1: axis 0 0 1 -> 0 0 -1

Commit message: updating rotation

File: mycobot_client_2/models/elephant_description/mycobot_280_pi.urdf (robot description, URDF)
Before this commit: robot firefighter, 10 links, 9 joints
Joints:
- joint joint2_to_joint1: axis 0 0 -1 -> 0 0 1; origin xyz=0 0 0.13956 rpy=0 0 0 -> xyz=0 0 -0.13956 rpy=3.141 0 0

Commit message: reverting urdf changes

File: mycobot_client_2/models/elephant_description/mycobot_280_pi.urdf (robot description, URDF)
Before this commit: robot firefighter, 10 links, 9 joints
Joints:
- joint joint2_to_joint1: origin xyz=0 0 -0.13956 rpy=3.141 0 0 -> xyz=0 0 0.13956 rpy=0 0 0

Commit message: Trying new urdf

File: mycobot_client_2/models/elephant_description/mycobot_280_pi.urdf (robot description, URDF)
Before this commit: robot firefighter, 10 links, 9 joints
Joints:
- joint joint2_to_joint1: axis 0 0 1 -> 0 0 -1

Commit message: adding visualizer

File: mycobot_client_2/models/elephant_description/mycobot_280_pi.urdf (robot description, URDF)
Before this commit: robot firefighter, 10 links, 9 joints
Joints:
- joint joint2_to_joint1: axis 0 0 -1 -> 0 0 1

Commit message: adding rotation of gripper

File: mycobot_client_2/models/elephant_description/mycobot_280_pi.urdf (robot description, URDF)
Before this commit: robot firefighter, 10 links, 9 joints
Joints:
- joint joint6output_to_gripper: origin xyz=0 0 0.1 rpy=0 0 0 -> xyz=0 0 0.1 rpy=0 0 -0.52

Commit message: updating urdf

File: mycobot_client_2/models/elephant_description/mycobot_280_pi.urdf (robot description, URDF)
Before this commit: robot firefighter, 10 links, 9 joints
Joints:
- joint joint6output_to_gripper: origin xyz=0 0 0.1 rpy=0 0 -0.52 -> xyz=0 0 0.1 rpy=0 0 0.52

Commit message: updating urdf, updating simple kinematics

File: mycobot_client_2/models/elephant_description/mycobot_280_pi.urdf (robot description, URDF)
Before this commit: robot firefighter, 10 links, 9 joints
Joints:
- joint joint6output_to_gripper: origin xyz=0 0 0.1 rpy=0 0 0.52 -> xyz=0 0 0.1 rpy=0 0 0.5236

Commit message: updating models

File: mycobot_client_2/models/elephant_description/mycobot_280_pi.urdf (robot description, URDF)
Before this commit: robot firefighter, 10 links, 9 joints
Joints:
- joint joint6output_to_gripper: origin xyz=0 0 0.1 rpy=0 0 0.5236 -> xyz=0 0 0.1 rpy=0 0 -0.5236

Commit message: Updating Docs, adding in Helper class (#6)
Adds documentation to the README on how to use this client package.
Adds documentation on the cobot client class
Adds an example script to run a task that students can modify
Adds an IK class that uses pybullet, not sim and control

File: mycobot_client_2/models/elephant_description/mycobot_280_pi.urdf (robot description, URDF)
Before this commit: robot firefighter, 10 links, 9 joints
Links:
- link g_base: mass 0.2 -> None; geometry 
Joints:
- joint g_base_to_joint1: origin xyz=0 0 0 rpy=0 0 0 -> xyz=0 0 0.026 rpy=0 0 0
- joint joint6output_to_gripper: origin xyz=0 0 0.12 rpy=0 0 0 -> xyz=0 0 0.1 rpy=0 0 -0.5236
- joint robot_base_to_g_base: origin xyz=0 0 0.12 rpy=0 0 0 -> xyz=0 0 0.003 rpy=0 0 0
